Commit message: fix: t265.stl bug & update doc

File: legged_perceptive_description/urdf/sensor_t265.xacro (robot description, xacro)
@@ -31,5 +31,5 @@
                 <origin xyz="0 0 0" rpy="0 0 0"/>
                 <geometry>
-                    <mesh filename="package://realsense2_description/meshes/t265.stl"/>
+                    <mesh filename="package://realsense2_description/meshes/d435.dae"/>
                 </geometry>
                 <material name="${name}_aluminum"/>
@@ -38,5 +38,5 @@
                 <origin xyz="0 0 0" rpy="0 0 0"/>
                 <geometry>
-                    <mesh filename="package://realsense2_description/meshes/t265.stl"/>
+                    <mesh filename="package://realsense2_description/meshes/d435.dae"/>
                 </geometry>
             </collision>
